Commit message: Use '' instead None for default value

File: test/component.urdf.xacro (robot description, xacro)
@@ -2,13 +2,11 @@
 <robot name="component" xmlns:xacro="http://wiki.ros.org/xacro">
   <link name="cover_link" />
-  <xacro:arg name="components_config_path" default="None" />
+  <xacro:arg name="components_config_path" default="''" />
   <xacro:property name="components_config_path_property" value="$(arg components_config_path)" />
-  <xacro:unless value="${components_config_path_property == 'None'}">
-    <xacro:include filename="$(find ros_components_description)/urdf/components.urdf.xacro"
-      ns="husarion_components" />
+  <xacro:if value="${components_config_path_property != ''}">
+    <xacro:include filename="$(find ros_components_description)/urdf/components.urdf.xacro" ns="husarion_components" />
     <xacro:husarion_components.create_components
       components_config_path="${components_config_path_property}"
-      namespace="None"
-    />
-  </xacro:unless>
+      namespace="" />
+  </xacro:if>
 </robot>

File: urdf/components.urdf.xacro (robot description, xacro)
@@ -1,8 +1,8 @@
 <?xml version="1.0" encoding="utf-8"?>
 <robot xmlns:xacro="http://wiki.ros.org/xacro">
-  <xacro:macro name="create_components"
-    params="components_config_path namespace">
-    <xacro:unless value="${components_config_path == 'None'}">
-      <xacro:property name="components_config"
+  <xacro:macro name="create_components" params="components_config_path namespace:=''">
+    <xacro:unless value="${components_config_path == ''}">
+      <xacro:property
+        name="components_config"
         value="${xacro.load_yaml(components_config_path)}" />
       <xacro:load_componenet
@@ -12,6 +12,5 @@
     </xacro:unless>
   </xacro:macro>
-  <xacro:macro name="load_componenet"
-    params="config counter robot_namespace">
+  <xacro:macro name="load_componenet" params="config counter robot_namespace:=''">
     <xacro:if value="${counter}">
       <xacro:property name="index" value="${counter - 1}" scope="parent" />
@@ -21,16 +20,6 @@
       <xacro:property name="xyz" value="${component['xyz']}" scope="parent" />
       <xacro:property name="rpy" value="${component['rpy']}" scope="parent" />
-      <xacro:if value="${robot_namespace == ''}">
-        <xacro:property name="ns" value="None" scope="parent" />
-      </xacro:if>
-      <xacro:unless value="${robot_namespace == ''}">
-        <xacro:property name="ns" value="${robot_namespace}" scope="parent" />
-      </xacro:unless>
-      <xacro:if value="${'device_namespace' in component}">
-        <xacro:property name="device_namespace" value="${component['device_namespace']}" scope="parent" />
-      </xacro:if>
-      <xacro:unless value="${'device_namespace' in component}">
-        <xacro:property name="device_namespace" value="" scope="parent" />
-      </xacro:unless>
+      <xacro:property name="ns" value="${robot_namespace}" scope="parent" />
+      <xacro:property name="device_ns" value="${component['device_namespace'] if 'device_namespace' in component else ''}" scope="parent" />
       <xacro:if value="${type == 'ANT02'}">
         <xacro:include
@@ -42,5 +31,5 @@
           rpy="${rpy}"
           namespace="${ns}"
-          device_namespace="${device_namespace}"
+          device_namespace="${device_ns}"
         />
       </xacro:if>
@@ -49,6 +38,6 @@
           filename="$(find ros_components_description)/urdf/orbbec_astra.urdf.xacro"
           ns="camera" />
-        <xacro:if value="${device_namespace == ''}">
-          <xacro:property name="device_namespace" value="camera" scope="parent" />
+        <xacro:if value="${device_ns == ''}">
+          <xacro:property name="device_ns" value="camera" scope="parent" />
         </xacro:if>
         <xacro:camera.orbbec_astra
@@ -57,5 +46,5 @@
           rpy="${rpy}"
           namespace="${ns}"
-          device_namespace="${device_namespace}"
+          device_namespace="${device_ns}"
         />
       </xacro:if>
@@ -70,6 +59,6 @@
           filename="$(find ros_components_description)/urdf/stereolabs_zed.urdf.xacro"
           ns="camera" />
-        <xacro:if value="${device_namespace == ''}">
-          <xacro:property name="device_namespace" value="zed" scope="parent" />
+        <xacro:if value="${device_ns == ''}">
+          <xacro:property name="device_ns" value="zed" scope="parent" />
         </xacro:if>
         <xacro:camera.zed_camera
@@ -78,5 +67,5 @@
           rpy="${rpy}"
           namespace="${ns}"
-          device_namespace="${device_namespace}"
+          device_namespace="${device_ns}"
           model="${zed_models_dict[type]}"
         />
@@ -97,5 +86,5 @@
           rpy="${rpy}"
           namespace="${ns}"
-          device_namespace="${device_namespace}"
+          device_namespace="${device_ns}"
           model="${rplidar_models_dict[type]}"
         />
@@ -120,5 +109,5 @@
           rpy="${rpy}"
           namespace="${ns}"
-          device_namespace="${device_namespace}"
+          device_namespace="${device_ns}"
           model="${ouster_models_dict[type]}"
         />
@@ -134,5 +123,5 @@
           rpy="${rpy}"
           namespace="${ns}"
-          device_namespace="${device_namespace}"
+          device_namespace="${device_ns}"
         />
       </xacro:if>
@@ -146,5 +135,5 @@
           xyz="${xyz}"
           rpy="${rpy}"
-          device_namespace="${device_namespace}"
+          device_namespace="${device_ns}"
           ur_type="ur3e"
         />
@@ -159,5 +148,5 @@
           xyz="${xyz}"
           rpy="${rpy}"
-          device_namespace="${device_namespace}"
+          device_namespace="${device_ns}"
           ur_type="ur5e"
         />
@@ -173,5 +162,5 @@
           rpy="${rpy}"
           namespace="${ns}"
-          device_namespace="${device_namespace}"
+          device_namespace="${device_ns}"
           kinova_type="gen3"
           dof="6"
@@ -190,5 +179,5 @@
           rpy="${rpy}"
           namespace="${ns}"
-          device_namespace="${device_namespace}"
+          device_namespace="${device_ns}"
           kinova_type="gen3"
           dof="6"
@@ -207,5 +196,5 @@
           rpy="${rpy}"
           namespace="${ns}"
-          device_namespace="${device_namespace}"
+          device_namespace="${device_ns}"
           kinova_type="gen3"
           dof="7"
@@ -228,5 +217,5 @@
           gripper="robotiq_2f_85"
           vision="true"
-          device_namespace="${device_namespace}"
+          device_namespace="${device_ns}"
         />
       </xacro:if>
@@ -239,5 +228,5 @@
           rpy="${rpy}"
           namespace="${ns}"
-          device_namespace="${device_namespace}"
+          device_namespace="${device_ns}"
           robotiq_type="2f_85"
         />
@@ -252,5 +241,5 @@
           rpy="${rpy}"
           namespace="${ns}"
-          device_namespace="${device_namespace}"
+          device_namespace="${device_ns}"
         />
       </xacro:if>

File: urdf/intel_realsense_d435.urdf.xacro (robot description, xacro)
@@ -18,14 +18,11 @@
 <robot name="intel_realsense_d435" xmlns:xacro="http://ros.org/wiki/xacro">
   <xacro:macro name="intel_realsense_d435"
-    params="parent_link xyz rpy
-            use_nominal_extrinsics:=false
-            namespace:=None
-            device_namespace:=camera">
-    <xacro:if value="${namespace == 'None'}">
-      <xacro:property name="ns" value="" />
-    </xacro:if>
-    <xacro:unless value="${namespace == 'None'}">
-        <xacro:property name="ns" value="${namespace}/" />
-    </xacro:unless>
+               params="parent_link
+                       xyz:='0.0 0.0 0.0'
+                       rpy:='0.0 0.0 0.0'
+                       use_nominal_extrinsics:=false
+                       namespace:=''
+                       device_namespace:=camera">
+    <xacro:property name="ns" value="${namespace + '/' if namespace != '' else ''}" />
     <!-- The following values are approximate, and the camera node
       publishing TF values with actual calibrated camera extrinsic values -->

File: urdf/kinova.urdf.xacro (robot description, xacro)
@@ -17,28 +17,19 @@
 <robot name="kinova" xmlns:xacro="http://ros.org/wiki/xacro">
   <xacro:macro name="kinova"
-    params="parent_link xyz rpy
-          kinova_type:=gen3_lite
-          dof:=6
-          gripper:=''
-          vision:=false
-          namespace:=None
-          device_namespace:=None
-          ">
+               params="parent_link
+                       xyz:='0.0 0.0 0.0'
+                       rpy:='0.0 0.0 0.0'
+                       kinova_type:=gen3_lite
+                       dof:=6
+                       gripper:=''
+                       vision:=false
+                       namespace:=''
+                       device_namespace:=''">
     <xacro:include
       filename="$(find kortex_description)/robots/kortex_robot.xacro"
       ns="kinova_manipulator"
     />
-    <xacro:if value="${namespace == 'None'}">
-      <xacro:property name="ns" value="" />
-    </xacro:if>
-    <xacro:unless value="${namespace == 'None'}">
-      <xacro:property name="ns" value="${namespace}/" />
-    </xacro:unless>
-    <xacro:if value="${device_namespace == ''}">
-      <xacro:property name="prefix" value="" />
-    </xacro:if>
-    <xacro:unless value="${device_namespace == ''}">
-      <xacro:property name="prefix" value="${device_namespace}_" />
-    </xacro:unless>
+    <xacro:property name="ns" value="${namespace + '/' if namespace != '' else ''}" />
+    <xacro:property name="prefix" value="${device_namespace + '_' if device_namespace != '' else ''}" />
     <!-- robot name parameter -->
     <xacro:property name="name" value="kinova_arm" />

File: urdf/orbbec_astra.urdf.xacro (robot description, xacro)
@@ -2,13 +2,10 @@
 <robot xmlns:xacro="http://www.ros.org/wiki/xacro">
   <xacro:macro name="orbbec_astra"
-               params="parent_link xyz rpy
-                       namespace:=None
+               params="parent_link
+                       xyz:='0.0 0.0 0.0'
+                       rpy:='0.0 0.0 0.0'
+                       namespace:=''
                        device_namespace:=camera">
-    <xacro:if value="${namespace == 'None'}">
-      <xacro:property name="ns" value="" />
-    </xacro:if>
-    <xacro:unless value="${namespace == 'None'}">
-      <xacro:property name="ns" value="${namespace}/" />
-    </xacro:unless>
+    <xacro:property name="ns" value="${namespace + '/' if namespace != '' else ''}" />
     <joint name="${parent_link.rstrip('_link')}_to_${device_namespace}_joint" type="fixed">
       <origin xyz="${xyz}" rpy="${rpy}" />

File: urdf/ouster.urdf.xacro (robot description, xacro)
@@ -2,8 +2,10 @@
 <robot xmlns:xacro="http://www.ros.org/wiki/xacro">
     <xacro:macro name="ouster"
-               params="parent_link xyz rpy
+               params="parent_link
+                       xyz:='0.0 0.0 0.0'
+                       rpy:='0.0 0.0 0.0'
                        model:=os1_32
-                       namespace:=None
-                       device_namespace:=None">
+                       namespace:=''
+                       device_namespace:=''">
     <xacro:if value="${model == 'os0_32'}">
       <xacro:property name="vfov" value="${radians(90.0)}" scope="parent" />
@@ -42,22 +44,6 @@
       <xacro:property name="mesh" value="ouster_os01" scope="parent"/>
     </xacro:if>
-    <xacro:if value="${namespace == 'None'}">
-      <xacro:property name="ns" value="" />
-    </xacro:if>
-    <xacro:unless value="${namespace == 'None'}">
-      <xacro:property name="ns" value="${namespace}/" />
-    </xacro:unless>
-    <xacro:if value="${device_namespace == ''}">
-      <xacro:property name="device_ns" value="" />
-    </xacro:if>
-    <xacro:unless value="${device_namespace == ''}">
-      <xacro:property name="device_ns" value="${device_namespace}/" />
-    </xacro:unless>
-    <xacro:if value="${device_namespace == ''}">
-      <xacro:property name="prefix" value="" />
-    </xacro:if>
-    <xacro:unless value="${device_namespace == ''}">
-      <xacro:property name="prefix" value="${device_namespace}_" />
-    </xacro:unless>
+    <xacro:property name="ns" value="${namespace + '/' if namespace != '' else ''}" />
+    <xacro:property name="prefix" value="${device_namespace + '_' if device_namespace != '' else ''}" />
     <joint name="${parent_link.rstrip('_link')}_to_${prefix}ouster_${model}_joint" type="fixed">
       <origin xyz="${xyz}" rpy="${rpy}" />
@@ -124,5 +110,5 @@
         </ray>
         <update_rate>20.0</update_rate>
-        <topic>${ns}${device_ns}ouster/points</topic>
+        <topic>${ns}${device_namespace}/ouster/points</topic>
         <frame_id>${ns}${prefix}os_lidar</frame_id>
         <gz_frame_id>${ns}${prefix}os_lidar</gz_frame_id>

File: urdf/robotiq.urdf.xacro (robot description, xacro)
@@ -17,18 +17,14 @@
 <robot name="robotiq" xmlns:xacro="http://ros.org/wiki/xacro">
   <xacro:macro name="robotiq"
-    params="parent_link xyz rpy
-            robotiq_type:=2f_85
-            namespace:=None
-            device_namespace:=None
-          ">
+               params="parent_link
+                       xyz:='0.0 0.0 0.0'
+                       rpy:='0.0 0.0 0.0'
+                       robotiq_type:=2f_85
+                       namespace:=''
+                       device_namespace:=''">
     <xacro:include
       filename="$(find robotiq_description)/urdf/robotiq_${robotiq_type}_macro.urdf.xacro"
       ns="gripper" />
-    <xacro:if value="${device_namespace == ''}">
-      <xacro:property name="prefix" value="" />
-    </xacro:if>
-    <xacro:unless value="${device_namespace == ''}">
-      <xacro:property name="prefix" value="${device_namespace}_" />
-    </xacro:unless>
+    <xacro:property name="prefix" value="${device_namespace + '_' if device_namespace != '' else ''}" />
     <xacro:gripper.robotiq_gripper name="${device_namespace}robotiq_${robotiq_type}"
       prefix="${prefix}"

File: urdf/slamtec_rplidar.urdf.xacro (robot description, xacro)
@@ -2,26 +2,12 @@
 <robot xmlns:xacro="http://www.ros.org/wiki/xacro">
   <xacro:macro name="slamtec_rplidar"
-               params="parent_link xyz rpy
-                       namespace:=None
-                       device_namespace:=None
+               params="parent_link
+                       xyz:='0.0 0.0 0.0'
+                       rpy:='0.0 0.0 0.0'
+                       namespace:=''
+                       device_namespace:=''
                        model:=s3">
-    <xacro:if value="${namespace == 'None'}">
-      <xacro:property name="ns" value="" />
-    </xacro:if>
-    <xacro:unless value="${namespace == 'None'}">
-      <xacro:property name="ns" value="${namespace}/" />
-    </xacro:unless>
-    <xacro:if value="${device_namespace == ''}">
-      <xacro:property name="device_ns" value="" />
-    </xacro:if>
-    <xacro:unless value="${device_namespace == ''}">
-      <xacro:property name="device_ns" value="${device_namespace}/" />
-    </xacro:unless>
-    <xacro:if value="${device_namespace == ''}">
-      <xacro:property name="prefix" value="" />
-    </xacro:if>
-    <xacro:unless value="${device_namespace == ''}">
-      <xacro:property name="prefix" value="${device_namespace}_" />
-    </xacro:unless>
+    <xacro:property name="ns" value="${namespace + '/' if namespace != '' else ''}" />
+    <xacro:property name="prefix" value="${device_namespace + '_' if device_namespace != '' else ''}" />
     <xacro:if value="${model == 's3'}">
       <!-- Spec: https://www.slamtec.ai/wp-content/uploads/2023/11/SLAMTEC_rplidar_datasheet_S3_v1.0_en.pdf -->
@@ -227,5 +213,5 @@
         <update_rate>10</update_rate>
         <visualize>false</visualize>
-        <topic>${ns}${device_ns}scan</topic>
+        <topic>${ns}${device_namespace}/scan</topic>
         <gz_frame_id>${ns}${prefix}laser</gz_frame_id>
         <ray>

File: urdf/stereolabs_zed.urdf.xacro (robot description, xacro)
@@ -19,14 +19,11 @@
   <xacro:property name="M_PI" value="3.1415926535897931" />
   <xacro:macro name="zed_camera"
-    params="parent_link xyz rpy
-    model:=zed
-    namespace:=None
-    device_namespace:=zed">
-    <xacro:if value="${namespace == 'None'}">
-      <xacro:property name="ns" value="" />
-    </xacro:if>
-    <xacro:unless value="${namespace == 'None'}">
-      <xacro:property name="ns" value="${namespace}/" />
-    </xacro:unless>
+               params="parent_link
+                       xyz:='0.0 0.0 0.0'
+                       rpy:='0.0 0.0 0.0'
+                       model:=zed
+                       namespace:=''
+                       device_namespace:=zed">
+    <xacro:property name="ns" value="${namespace + '/' if namespace != '' else ''}" />
     <xacro:if value="${model == 'zed'}">
       <xacro:property name="baseline" value="0.12" />

File: urdf/teltonika_003R-00253.urdf.xacro (robot description, xacro)
@@ -1,15 +1,11 @@
 <?xml version="1.0" encoding="utf-8"?>
 <robot xmlns:xacro="http://wiki.ros.org/xacro">
-  <xacro:macro
-    name="teltonika_003R-00253"
-    params="parent_link xyz rpy
-            namespace:=None
-            device_namespace:=gps">
-    <xacro:if value="${namespace == 'None'}">
-      <xacro:property name="ns" value="" />
-    </xacro:if>
-    <xacro:unless value="${namespace == 'None'}">
-      <xacro:property name="ns" value="${namespace}/" />
-    </xacro:unless>
+  <xacro:macro name="teltonika_003R-00253"
+               params="parent_link
+                       xyz:='0.0 0.0 0.0'
+                       rpy:='0.0 0.0 0.0'
+                       namespace:=''
+                       device_namespace:=gps">
+    <xacro:property name="ns" value="${namespace + '/' if namespace != '' else ''}" />
     <joint name="${parent_link.rstrip('_link')}_to_antenna_joint"
       type="fixed">

File: urdf/ur.urdf.xacro (robot description, xacro)
@@ -17,17 +17,11 @@
 <robot name="ur" xmlns:xacro="http://ros.org/wiki/xacro">
   <xacro:macro name="ur"
-    params="parent_link xyz rpy
-          device_namespace:=None
-          ur_type:=ur3e">
-    <xacro:include
-      filename="$(find ur_description)/urdf/ur_macro.xacro"
-      ns="ur_manipulator"
-    />
-    <xacro:if value="${device_namespace == ''}">
-      <xacro:property name="prefix" value="" />
-    </xacro:if>
-    <xacro:unless value="${device_namespace == ''}">
-      <xacro:property name="prefix" value="${device_namespace}_" />
-    </xacro:unless>
+               params="parent_link
+                       xyz:='0.0 0.0 0.0'
+                       rpy:='0.0 0.0 0.0'
+                       device_namespace:=''
+                       ur_type:=ur3e">
+    <xacro:include filename="$(find ur_description)/urdf/ur_macro.xacro" ns="ur_manipulator" />
+    <xacro:property name="prefix" value="${device_namespace + '_' if device_namespace != '' else ''}" />
     <xacro:property name="joint_limit_params"
       value="$(find ur_description)/config/${ur_type}/joint_limits.yaml" scope="parent" />
@@ -51,6 +45,4 @@
       physical_parameters_file="${physical_params}"
       visual_parameters_file="${visual_params}"
-      sim_ignition="true"
-      generate_ros2_control_tag="false"
     >
       <origin xyz="${xyz}" rpy="${rpy}" />

File: urdf/velodyne_puck.urdf.xacro (robot description, xacro)
@@ -2,25 +2,11 @@
 <robot xmlns:xacro="http://www.ros.org/wiki/xacro">
   <xacro:macro name="velodyne_puck"
-               params="parent_link xyz rpy
-                       namespace:=None
-                       device_namespace:=None">
-    <xacro:if value="${namespace == 'None'}">
-      <xacro:property name="ns" value="" />
-    </xacro:if>
-    <xacro:unless value="${namespace == 'None'}">
-      <xacro:property name="ns" value="${namespace}/" />
-    </xacro:unless>
-    <xacro:if value="${device_namespace == ''}">
-      <xacro:property name="device_ns" value="" />
-    </xacro:if>
-    <xacro:unless value="${device_namespace == ''}">
-      <xacro:property name="device_ns" value="${device_namespace}/" />
-    </xacro:unless>
-    <xacro:if value="${device_namespace == ''}">
-      <xacro:property name="prefix" value="" />
-    </xacro:if>
-    <xacro:unless value="${device_namespace == ''}">
-      <xacro:property name="prefix" value="${device_namespace}_" />
-    </xacro:unless>
+               params="parent_link
+                       xyz:='0.0 0.0 0.0'
+                       rpy:='0.0 0.0 0.0'
+                       namespace:=''
+                       device_namespace:=''">
+    <xacro:property name="ns" value="${namespace + '/' if namespace != '' else ''}" />
+    <xacro:property name="prefix" value="${device_namespace + '_' if device_namespace != '' else ''}" />
     <joint name="${parent_link.rstrip('_link')}_to_${prefix}velodyne_puck_joint" type="fixed">
       <origin xyz="${xyz}" rpy="${rpy}" />
@@ -88,5 +74,5 @@
           </noise>
         </ray>
-        <topic>${ns}${device_ns}velodyne_points</topic>
+        <topic>${ns}${device_namespace}/velodyne_points</topic>
         <frame_id>${ns}${prefix}velodyne</frame_id>
         <gz_frame_id>${ns}${prefix}velodyne</gz_frame_id>

File: urdf/wibotic_receiver.urdf.xacro (robot description, xacro)
@@ -17,25 +17,11 @@
 <robot xmlns:xacro="http://www.ros.org/wiki/xacro">
   <xacro:macro name="wibotic_receiver"
-    params="parent_link xyz rpy
-                         namespace:=None
-                          device_namespace:=None">
-    <xacro:if value="${namespace == 'None'}">
-      <xacro:property name="ns" value="" />
-    </xacro:if>
-    <xacro:unless value="${namespace == 'None'}">
-      <xacro:property name="ns" value="${namespace}/" />
-    </xacro:unless>
-    <xacro:if value="${device_namespace == ''}">
-      <xacro:property name="device_ns" value="" />
-    </xacro:if>
-    <xacro:unless value="${device_namespace == ''}">
-      <xacro:property name="device_ns" value="${device_namespace}/" />
-    </xacro:unless>
-    <xacro:if value="${device_namespace == ''}">
-      <xacro:property name="prefix" value="" />
-    </xacro:if>
-    <xacro:unless value="${device_namespace == ''}">
-      <xacro:property name="prefix" value="${device_namespace}_" />
-    </xacro:unless>
+               params="parent_link
+                       xyz:='0.0 0.0 0.0'
+                       rpy:='0.0 0.0 0.0'
+                       namespace:=''
+                       device_namespace:=''">
+    <xacro:property name="ns" value="${namespace + '/' if namespace != '' else ''}" />
+    <xacro:property name="prefix" value="${device_namespace + '_' if device_namespace != '' else ''}" />
     <joint name="${parent_link.rstrip('_link')}_to_${prefix}wibotic_receiver_joint" type="fixed">
       <origin xyz="${xyz}" rpy="${rpy}" />
