Commit message: Simplify

File: urdf/slamtec_rplidar.urdf.xacro (robot description, xacro)
@@ -17,5 +17,5 @@
       <xacro:property name="dist_res" value="0.01" />
       <xacro:property name="std_dev" value="0.03" />
-      <xacro:property name="mesh" value="slamtec_rplidar_s3.dae" />
+      <xacro:property name="mesh" value="s3.dae" />
       <xacro:property name="collision">
         <origin xyz="0.0 0.0 ${0.0413/2.0}" rpy="0.0 0.0 0.0" />
@@ -42,5 +42,5 @@
       <xacro:property name="dist_res" value="0.013" />
       <xacro:property name="std_dev" value="0.03" />
-      <xacro:property name="mesh" value="slamtec_rplidar_s2.dae" />
+      <xacro:property name="mesh" value="s2.dae" />
       <xacro:property name="collision">
         <origin xyz="0.0 0.0 ${0.038857/2.0}" rpy="0.0 0.0 0.0" />
@@ -67,5 +67,5 @@
       <xacro:property name="dist_res" value="0.03" />
       <xacro:property name="std_dev" value="0.05" />
-      <xacro:property name="mesh" value="slamtec_rplidar_s1.dae" />
+      <xacro:property name="mesh" value="s1.dae" />
       <xacro:property name="collision">
         <origin xyz="0.0 0.0 ${0.0195/2.0}" rpy="0.0 0.0 0.0" />
@@ -92,5 +92,5 @@
       <xacro:property name="dist_res" value="0.03" />
       <xacro:property name="std_dev" value="0.05" />
-      <xacro:property name="mesh" value="slamtec_rplidar_ax.dae" />
+      <xacro:property name="mesh" value="ax.dae" />
       <xacro:property name="collision">
         <origin xyz="0.0 0.0 ${0.041/2.0}" rpy="0.0 0.0 0.0" />
@@ -117,5 +117,5 @@
       <xacro:property name="dist_res" value="0.03" />
       <xacro:property name="std_dev" value="0.05" />
-      <xacro:property name="mesh" value="slamtec_rplidar_ax.dae" />
+      <xacro:property name="mesh" value="ax.dae" />
       <xacro:property name="collision">
         <origin xyz="0.0 0.0 ${0.041/2.0}" rpy="0.0 0.0 0.0" />
@@ -141,5 +141,5 @@
       <xacro:property name="dist_res" value="0.03" />
       <xacro:property name="std_dev" value="0.05" />
-      <xacro:property name="mesh" value="slamtec_rplidar_a2m8.dae" />
+      <xacro:property name="mesh" value="a2m8.dae" />
       <xacro:property name="collision">
         <origin xyz="0.0 0.0 ${0.041/2.0}" rpy="0.0 0.0 0.0" />
@@ -165,5 +165,5 @@
       <xacro:property name="dist_res" value="0.03" />
       <xacro:property name="std_dev" value="0.05" />
-      <xacro:property name="mesh" value="slamtec_rplidar_ax.dae" />
+      <xacro:property name="mesh" value="ax.dae" />
       <xacro:property name="collision">
         <origin xyz="0.0 0.0 ${0.041/2.0}" rpy="0.0 0.0 0.0" />
@@ -192,5 +192,5 @@
         <origin xyz="0.0 0.0 0.0" rpy="0.0 0.0 0.0" />
         <geometry>
-          <mesh filename="package://ros_components_description/meshes/${mesh}" />
+          <mesh filename="package://ros_components_description/meshes/rplidar/${mesh}" />
         </geometry>
       </visual>

File: urdf/ur.urdf.xacro (robot description, xacro)
@@ -50,5 +50,5 @@
     <ros2_control name="${prefix + ur_type}" type="system">
       <hardware>
-        <plugin>ign_ros2_control/IgnitionSystem</plugin>
+        <plugin>gz_ros2_control/GazeboSimSystem</plugin>
       </hardware>
       <joint name="${prefix}shoulder_pan_joint">

Commit message: Fix Rplidar S1 colission

File: urdf/slamtec_rplidar.urdf.xacro (robot description, xacro)
@@ -69,6 +69,7 @@
       <xacro:property name="mesh" value="s1.dae" />
       <xacro:property name="collision">
-        <origin xyz="0.0 0.0 ${0.0195/2.0}" rpy="0.0 0.0 0.0" />
-        <geometry>
+        <origin xyz="0.0 0.0 0.025" rpy="0.0 0.0 0.0" />
+        <geometry>
+          <cylinder radius="0.022" length="0.05" />
           <box size="0.0555 0.0555 0.0195" />
         </geometry>

Commit message: Accuracy is 2 * std_dev

File: urdf/slamtec_rplidar.urdf.xacro (robot description, xacro)
@@ -16,5 +16,5 @@
       <xacro:property name="dist_max" value="40.0" />
       <xacro:property name="dist_res" value="0.01" />
-      <xacro:property name="std_dev" value="0.03" />
+      <xacro:property name="std_dev" value="0.015" />
       <xacro:property name="mesh" value="s3.dae" />
       <xacro:property name="collision">
@@ -41,5 +41,5 @@
       <xacro:property name="dist_max" value="30.0" />
       <xacro:property name="dist_res" value="0.013" />
-      <xacro:property name="std_dev" value="0.03" />
+      <xacro:property name="std_dev" value="0.015" />
       <xacro:property name="mesh" value="s2.dae" />
       <xacro:property name="collision">
@@ -66,5 +66,5 @@
       <xacro:property name="dist_max" value="40.0" />
       <xacro:property name="dist_res" value="0.03" />
-      <xacro:property name="std_dev" value="0.05" />
+      <xacro:property name="std_dev" value="0.025" />
       <xacro:property name="mesh" value="s1.dae" />
       <xacro:property name="collision">
