Commit message: Fix tests

File: urdf/dev.urdf.xacro (robot description, xacro)
@@ -3,10 +3,5 @@
   <xacro:macro name="dev"
                params="namespace:=None model:=dev01">
-    <xacro:if value="${namespace == 'None'}">
-      <xacro:property name="ns" value="" />
-    </xacro:if>
-    <xacro:unless value="${namespace == 'None'}">
-      <xacro:property name="ns" value="${namespace}/" />
-    </xacro:unless>
+    <xacro:property name="ns" value="${namespace + '/' if namespace != '' else ''}" />
     <xacro:if value="${model == 'dev01'}">
       <xacro:property name="parent_link" value="base_link" scope="parent" />

Commit message: fix links

File: urdf/dev.urdf.xacro (robot description, xacro)
@@ -10,5 +10,5 @@
     </xacro:unless>
     <xacro:if value="${model == 'dev01'}">
-      <xacro:property name="parent_link" value="base_link" scope="parent" />
+      <xacro:property name="parent_link" value="body_link" scope="parent" />
       <!-- 0.0001 in z is to cover the base. -->
       <xacro:property name="xyz" value="0 0 0.0001"  scope="parent" />
@@ -20,5 +20,5 @@
     </xacro:if>
     <xacro:if value="${model == 'dev02'}">
-      <xacro:property name="parent_link" value="base_link" scope="parent" />
+      <xacro:property name="parent_link" value="body_link" scope="parent" />
       <xacro:property name="xyz" value="0 0 0"  scope="parent" />
       <xacro:property name="rpy" value="0 0 ${-pi/2.0}" scope="parent" />
@@ -28,5 +28,5 @@
     </xacro:if>
     <xacro:if value="${model == 'dev03'}">
-      <xacro:property name="parent_link" value="base_link" scope="parent" />
+      <xacro:property name="parent_link" value="body_link" scope="parent" />
       <xacro:property name="xyz" value="0 0 0"  scope="parent" />
       <xacro:property name="rpy" value="0 0 ${-pi/2.0}" scope="parent" />
@@ -36,5 +36,5 @@
     </xacro:if>
     <xacro:if value="${model == 'dev04l'}">
-      <xacro:property name="parent_link" value="base_link" scope="parent" />
+      <xacro:property name="parent_link" value="body_link" scope="parent" />
       <xacro:property name="xyz" value="0 0 0"  scope="parent" />
       <xacro:property name="rpy" value="0 0 ${-pi/2.0}" scope="parent" />
@@ -44,5 +44,5 @@
     </xacro:if>
     <xacro:if value="${model == 'dev04h'}">
-      <xacro:property name="parent_link" value="base_link" scope="parent" />
+      <xacro:property name="parent_link" value="body_link" scope="parent" />
       <xacro:property name="xyz" value="0 0 0"  scope="parent" />
       <xacro:property name="rpy" value="0 0 ${-pi/2.0}" scope="parent" />
@@ -55,10 +55,10 @@
       <xacro:property name="xyz" value="-0.185 0 0"  scope="parent" />
       <xacro:property name="rpy" value="0 0 ${-pi/2.0}" scope="parent" />
-      <xacro:property name="collision_box_size" value="0.028 0.12 0.35"      scope="parent" />
+      <xacro:property name="collision_box_size" value="0.028 0.04 0.35"      scope="parent" />
       <xacro:property name="collision_box_rpy"  value="0 0 ${-pi/2.0}"      scope="parent" />
       <xacro:property name="collision_box_xyz"  value="0 0 0.175"      scope="parent" />
     </xacro:if>
     <xacro:if value="${model == 'dev06'}">
-      <xacro:property name="parent_link" value="base_link" scope="parent" />
+      <xacro:property name="parent_link" value="body_link" scope="parent" />
       <xacro:property name="xyz" value="0 0 0"  scope="parent" />
       <xacro:property name="rpy" value="0 0 ${-pi/2.0}" scope="parent" />
@@ -71,5 +71,5 @@
       <xacro:property name="xyz" value="0 0 0"  scope="parent" />
       <xacro:property name="rpy" value="0 0 ${-pi/2.0}" scope="parent" />
-      <xacro:property name="collision_box_size" value="0.175 0.525 0.14"      scope="parent" />
+      <xacro:property name="collision_box_size" value="0.175 0.525 0.143"      scope="parent" />
       <xacro:property name="collision_box_rpy"  value="0 0 ${-pi/2.0}"      scope="parent" />
       <xacro:property name="collision_box_xyz"  value="0 0 0.07"      scope="parent" />
@@ -79,5 +79,5 @@
       <xacro:property name="xyz" value="0 0 0"  scope="parent" />
       <xacro:property name="rpy" value="0 0 0" scope="parent" />
-      <xacro:property name="collision_box_size" value="0.175 0.4 0.14"      scope="parent" />
+      <xacro:property name="collision_box_size" value="0.175 0.4 0.143"      scope="parent" />
       <xacro:property name="collision_box_rpy"  value="0 0 ${-pi/2.0}"      scope="parent" />
       <xacro:property name="collision_box_xyz"  value="0 0 0.07"      scope="parent" />
