Commit message: Removed None from device_namespace (#58)
* Removed None from device_namespace, allow to not declare device_namespace inside yaml

Signed-off-by: Jakub Delicat <jakub.delicat@husarion.com>

* Fixed launch errorrs

Signed-off-by: Jakub Delicat <jakub.delicat@husarion.com>

* Delete empty line

---------

Signed-off-by: Jakub Delicat <jakub.delicat@husarion.com>
Co-authored-by: rafal-gorecki <rafal.gorecki@husarion.com>

File: urdf/components.urdf.xacro (robot description, xacro)
@@ -21,6 +21,4 @@
       <xacro:property name="xyz" value="${component['xyz']}" scope="parent" />
       <xacro:property name="rpy" value="${component['rpy']}" scope="parent" />
-      <xacro:property name="device_namespace" value="${component['device_namespace']}"
-        scope="parent" />
       <xacro:if value="${robot_namespace == ''}">
         <xacro:property name="ns" value="None" scope="parent" />
@@ -29,4 +27,10 @@
         <xacro:property name="ns" value="${robot_namespace}" scope="parent" />
       </xacro:unless>
+      <xacro:if value="${'device_namespace' in component}">
+        <xacro:property name="device_namespace" value="${component['device_namespace']}" scope="parent" />
+      </xacro:if>
+      <xacro:unless value="${'device_namespace' in component}">
+        <xacro:property name="device_namespace" value="" scope="parent" />
+      </xacro:unless>
       <xacro:if value="${type == 'ANT02'}">
         <xacro:include
@@ -45,4 +49,7 @@
           filename="$(find ros_components_description)/urdf/orbbec_astra.urdf.xacro"
           ns="camera" />
+        <xacro:if value="${device_namespace == ''}">
+          <xacro:property name="device_namespace" value="camera" scope="parent" />
+        </xacro:if>
         <xacro:camera.orbbec_astra
           parent_link="${parent_link}"
@@ -63,4 +70,7 @@
           filename="$(find ros_components_description)/urdf/stereolabs_zed.urdf.xacro"
           ns="camera" />
+        <xacro:if value="${device_namespace == ''}">
+          <xacro:property name="device_namespace" value="zed" scope="parent" />
+        </xacro:if>
         <xacro:camera.zed_camera
           parent_link="${parent_link}"

File: urdf/kinova.urdf.xacro (robot description, xacro)
@@ -35,8 +35,8 @@
       <xacro:property name="ns" value="${namespace}/" />
     </xacro:unless>
-    <xacro:if value="${device_namespace == 'None'}">
+    <xacro:if value="${device_namespace == ''}">
       <xacro:property name="prefix" value="" />
     </xacro:if>
-    <xacro:unless value="${device_namespace == 'None'}">
+    <xacro:unless value="${device_namespace == ''}">
       <xacro:property name="prefix" value="${device_namespace}_" />
     </xacro:unless>

File: urdf/ouster.urdf.xacro (robot description, xacro)
@@ -48,14 +48,14 @@
       <xacro:property name="ns" value="${namespace}/" />
     </xacro:unless>
-    <xacro:if value="${device_namespace == 'None'}">
+    <xacro:if value="${device_namespace == ''}">
       <xacro:property name="device_ns" value="" />
     </xacro:if>
-    <xacro:unless value="${device_namespace == 'None'}">
+    <xacro:unless value="${device_namespace == ''}">
       <xacro:property name="device_ns" value="${device_namespace}/" />
     </xacro:unless>
-    <xacro:if value="${device_namespace == 'None'}">
+    <xacro:if value="${device_namespace == ''}">
       <xacro:property name="prefix" value="" />
     </xacro:if>
-    <xacro:unless value="${device_namespace == 'None'}">
+    <xacro:unless value="${device_namespace == ''}">
       <xacro:property name="prefix" value="${device_namespace}_" />
     </xacro:unless>

File: urdf/robotiq.urdf.xacro (robot description, xacro)
@@ -25,8 +25,8 @@
       filename="$(find robotiq_description)/urdf/robotiq_${robotiq_type}_macro.urdf.xacro"
       ns="gripper" />
-    <xacro:if value="${device_namespace == 'None'}">
+    <xacro:if value="${device_namespace == ''}">
       <xacro:property name="prefix" value="" />
     </xacro:if>
-    <xacro:unless value="${device_namespace == 'None'}">
+    <xacro:unless value="${device_namespace == ''}">
       <xacro:property name="prefix" value="${device_namespace}_" />
     </xacro:unless>

File: urdf/slamtec_rplidar.urdf.xacro (robot description, xacro)
@@ -12,14 +12,14 @@
       <xacro:property name="ns" value="${namespace}/" />
     </xacro:unless>
-    <xacro:if value="${device_namespace == 'None'}">
+    <xacro:if value="${device_namespace == ''}">
       <xacro:property name="device_ns" value="" />
     </xacro:if>
-    <xacro:unless value="${device_namespace == 'None'}">
+    <xacro:unless value="${device_namespace == ''}">
       <xacro:property name="device_ns" value="${device_namespace}/" />
     </xacro:unless>
-    <xacro:if value="${device_namespace == 'None'}">
+    <xacro:if value="${device_namespace == ''}">
       <xacro:property name="prefix" value="" />
     </xacro:if>
-    <xacro:unless value="${device_namespace == 'None'}">
+    <xacro:unless value="${device_namespace == ''}">
       <xacro:property name="prefix" value="${device_namespace}_" />
     </xacro:unless>

File: urdf/ur.urdf.xacro (robot description, xacro)
@@ -24,8 +24,8 @@
       ns="ur_manipulator"
     />
-    <xacro:if value="${device_namespace == 'None'}">
+    <xacro:if value="${device_namespace == ''}">
       <xacro:property name="prefix" value="" />
     </xacro:if>
-    <xacro:unless value="${device_namespace == 'None'}">
+    <xacro:unless value="${device_namespace == ''}">
       <xacro:property name="prefix" value="${device_namespace}_" />
     </xacro:unless>

File: urdf/velodyne_puck.urdf.xacro (robot description, xacro)
@@ -11,14 +11,14 @@
       <xacro:property name="ns" value="${namespace}/" />
     </xacro:unless>
-    <xacro:if value="${device_namespace == 'None'}">
+    <xacro:if value="${device_namespace == ''}">
       <xacro:property name="device_ns" value="" />
     </xacro:if>
-    <xacro:unless value="${device_namespace == 'None'}">
+    <xacro:unless value="${device_namespace == ''}">
       <xacro:property name="device_ns" value="${device_namespace}/" />
     </xacro:unless>
-    <xacro:if value="${device_namespace == 'None'}">
+    <xacro:if value="${device_namespace == ''}">
       <xacro:property name="prefix" value="" />
     </xacro:if>
-    <xacro:unless value="${device_namespace == 'None'}">
+    <xacro:unless value="${device_namespace == ''}">
       <xacro:property name="prefix" value="${device_namespace}_" />
     </xacro:unless>

File: urdf/wibotic_receiver.urdf.xacro (robot description, xacro)
@@ -26,14 +26,14 @@
       <xacro:property name="ns" value="${namespace}/" />
     </xacro:unless>
-    <xacro:if value="${device_namespace == 'None'}">
+    <xacro:if value="${device_namespace == ''}">
       <xacro:property name="device_ns" value="" />
     </xacro:if>
-    <xacro:unless value="${device_namespace == 'None'}">
+    <xacro:unless value="${device_namespace == ''}">
       <xacro:property name="device_ns" value="${device_namespace}/" />
     </xacro:unless>
-    <xacro:if value="${device_namespace == 'None'}">
+    <xacro:if value="${device_namespace == ''}">
       <xacro:property name="prefix" value="" />
     </xacro:if>
-    <xacro:unless value="${device_namespace == 'None'}">
+    <xacro:unless value="${device_namespace == ''}">
       <xacro:property name="prefix" value="${device_namespace}_" />
     </xacro:unless>

Commit message: Add use_sim arg

File: urdf/components.urdf.xacro (robot description, xacro)
@@ -1,5 +1,5 @@
 <?xml version="1.0" encoding="utf-8"?>
 <robot xmlns:xacro="http://wiki.ros.org/xacro">
-  <xacro:macro name="create_components" params="components_config_path namespace:=''">
+  <xacro:macro name="create_components" params="components_config_path namespace:='' use_sim:='False'">
     <xacro:unless value="${components_config_path == ''}">
       <xacro:property
@@ -71,4 +71,21 @@
         />
       </xacro:if>
+      <xacro:if value="${type == 'CAM11'}">
+        <xacro:include
+          filename="$(find ros_components_description)/urdf/luxonis_depthai.urdf.xacro"
+          ns="camera" />
+        <xacro:if value="${device_ns == ''}">
+          <xacro:property name="device_ns" value="camera" scope="parent" />
+        </xacro:if>
+        <xacro:camera.luxonis_depthai
+          parent_link="${parent_link}"
+          xyz="${xyz}"
+          rpy="${rpy}"
+          namespace="${ns}"
+          device_namespace="${device_ns}"
+          model="OAK-D-PRO"
+          use_sim="${use_sim}"
+        />
+      </xacro:if>
       <xacro:property name="rplidar_models_dict"
         value="${dict ([

Commit message: Simulate luxonis OAK

File: urdf/components.urdf.xacro (robot description, xacro)
@@ -76,5 +76,5 @@
           ns="camera" />
         <xacro:if value="${device_ns == ''}">
-          <xacro:property name="device_ns" value="camera" scope="parent" />
+          <xacro:property name="device_ns" value="oak" scope="parent" />
         </xacro:if>
         <xacro:camera.luxonis_depthai

File: urdf/luxonis_depthai.urdf.xacro (robot description, xacro)
@@ -6,14 +6,36 @@
                        rpy:='0.0 0.0 0.0'
                        namespace:=''
-                       device_namespace:=oak
-                       model:=OAK-D-PRO
+                       device_namespace:='oak'
+                       model:='OAK-D-PRO'
                        use_sim:=False">
 	<xacro:include filename="$(find depthai_descriptions)/urdf/include/depthai_macro.urdf.xacro" />
   <xacro:property name="ns" value="${namespace + '/' if namespace != '' else ''}" />
 	<xacro:depthai_camera camera_name="${ns}${device_namespace}" parent="${parent_link}"
-  	base_frame="oak-d_frame" camera_model="${model}"
+  	base_frame="${ns}${device_namespace}" camera_model="${model}"
 		cam_pos_x="${xyz.split()[0]}" cam_pos_y="${xyz.split()[1]}" cam_pos_z="${xyz.split()[2]}"
 		cam_roll="${rpy.split()[0]}" cam_pitch="${rpy.split()[1]}" cam_yaw="${rpy.split()[2]}"
     simulation="${use_sim}" />
+  <xacro:include filename="$(find ros_components_description)/urdf/gz_sensor.urdf.xacro" ns="gz_sensor" />
+  <xacro:gz_sensor.camera
+    reference="${ns}${device_namespace}"
+    name="${ns}${device_namespace}_color"
+    topic="${ns}${device_namespace}/rgb/color"
+    frame_id="${ns}${device_namespace}_rgb_camera_frame"
+    frequency="30"
+    width="1280"
+    height="720"
+    fov="${60.0/180.0*pi}" />
+  <xacro:gz_sensor.depth_camera
+    reference="${ns}${device_namespace}"
+    name="${ns}${device_namespace}_depth"
+    topic="${ns}${device_namespace}/stereo/depth"
+    frame_id="${ns}${device_namespace}_rgb_camera_frame"
+    frequency="30"
+    width="1280"
+    height="720"
+    fov="${60.0/180.0*pi}"
+    min_dist="1.0"
+    max_dist="12.0"
+    stddev_error="0.2" />
   </xacro:macro>
 </robot>

File: urdf/orbbec_astra.urdf.xacro (robot description, xacro)
@@ -72,46 +72,28 @@
     </joint>
     <link name="${device_namespace}_color_optical_frame" />
-    <gazebo reference="${device_namespace}_link">
-      <!-- https://github.com/orbbec/OrbbecSDK_ROS2#all-available-topics -->
-      <sensor type="camera" name="${ns}${device_namespace}_orbbec_astra_color">
-        <always_on>true</always_on>
-        <update_rate>30.0</update_rate>
-        <topic>${ns}${device_namespace}/color/image_raw</topic>
-        <visualize>false</visualize>
-        <gz_frame_id>${ns}${device_namespace}_color_optical_frame</gz_frame_id>
-        <horizontal_fov>${60.0/180.0*pi}</horizontal_fov>
-        <image>
-          <width>640</width>
-          <height>480</height>
-        </image>
-        <clip>
-          <near>0.6</near>
-          <far>8.0</far>
-        </clip>
-      </sensor>
-      <sensor type="depth_camera" name="${ns}${device_namespace}_orbbec_astra_depth">
-        <always_on>true</always_on>
-        <update_rate>10.0</update_rate>
-        <topic>${ns}${device_namespace}/depth/image_raw</topic>
-        <visualize>false</visualize>
-        <gz_frame_id>${ns}${device_namespace}_depth_optical_frame</gz_frame_id>
-        <camera>
-          <horizontal_fov>${60.0/180.0*pi}</horizontal_fov>
-          <image>
-            <width>640</width>
-            <height>480</height>
-          </image>
-          <clip>
-            <near>0.6</near>
-            <far>8.0</far>
-          </clip>
-          <noise>
-            <type>gaussian</type>
-            <mean>0.0</mean>
-            <stddev>0.005</stddev>
-          </noise>
-        </camera>
-      </sensor>
-    </gazebo>
+    <!-- GAZEBO -->
+    <!-- https://github.com/orbbec/OrbbecSDK_ROS2#all-available-topics -->
+    <xacro:include filename="$(find ros_components_description)/urdf/gz_sensor.urdf.xacro" ns="gz_sensor" />
+    <xacro:gz_sensor.camera
+      reference="${device_namespace}_link"
+      name="${ns}${device_namespace}_orbbec_astra_color"
+      topic="${ns}${device_namespace}/color/image_raw"
+      frame_id="${ns}${device_namespace}_color_optical_frame"
+      frequency="30"
+      width="640"
+      height="480"
+      fov="${60.0/180.0*pi}" />
+    <xacro:gz_sensor.depth_camera
+      reference="${device_namespace}_link"
+      name="${ns}${device_namespace}_orbbec_astra_depth"
+      topic="${ns}${device_namespace}/depth/image_raw"
+      frame_id="${ns}${device_namespace}_depth_optical_frame"
+      frequency="30"
+      width="640"
+      height="480"
+      fov="${60.0/180.0*pi}"
+      min_dist="0.6"
+      max_dist="8.0"
+      stddev_error="0.05" />
   </xacro:macro>
 </robot>

Commit message: Ros2 fix camera resolution (#61)
* fix camera resolution

* all CAM02 launch

* add use_sim arg

* add depth points

File: urdf/components.urdf.xacro (robot description, xacro)
@@ -2,5 +2,5 @@
 <robot xmlns:xacro="http://wiki.ros.org/xacro">
   <xacro:macro name="create_components"
-    params="components_config_path namespace">
+    params="components_config_path namespace use_sim:=false">
     <xacro:unless value="${components_config_path == 'None'}">
       <xacro:property name="components_config"
@@ -9,9 +9,10 @@
         config="${components_config}"
         counter="${len(components_config['components'])}"
-        robot_namespace="${namespace}" />
+        robot_namespace="${namespace}"
+        use_sim="${use_sim}" />
     </xacro:unless>
   </xacro:macro>
   <xacro:macro name="load_componenet"
-    params="config counter robot_namespace">
+    params="config counter robot_namespace use_sim:=false">
     <xacro:if value="${counter}">
       <xacro:property name="index" value="${counter - 1}" scope="parent" />
@@ -84,4 +85,20 @@
           />
         </xacro:if>
+        <xacro:if value="${type == 'CAM02'}">
+          <xacro:include
+            filename="$(find ros_components_description)/urdf/intel_realsense_d435.urdf.xacro"
+            ns="camera" />
+          <xacro:if value="${device_namespace == ''}">
+            <xacro:property name="device_namespace" value="camera" scope="parent" />
+          </xacro:if>
+          <xacro:camera.intel_realsense_d435
+            parent_link="${parent_link}"
+            xyz="${xyz}"
+            rpy="${rpy}"
+            namespace="${ns}"
+            device_namespace="${device_namespace}"
+            use_nominal_extrinsics="${use_sim}"
+          />
+        </xacro:if>
         <xacro:property name="zed_models_dict"
           value="${dict ([

Commit message: Add configurations

File: urdf/components.urdf.xacro (robot description, xacro)
@@ -114,5 +114,10 @@
           />
         </xacro:if>
-        <xacro:if value="${type == 'CAM11'}">
+        <!-- 'CAM10', 'OAK-1-LITE' is not available in luxonis repo -->
+        <xacro:property name="luxonis_models_dict"
+          value="${dict ([
+          ('CAM11', 'OAK-D-PRO'),
+          ])}" />
+        <xacro:if value="${type in luxonis_models_dict}">
           <xacro:include
             filename="$(find ros_components_description)/urdf/luxonis_depthai.urdf.xacro"
@@ -127,5 +132,5 @@
             namespace="${ns}"
             device_namespace="${device_ns}"
-            model="OAK-D-PRO"
+            model="${luxonis_models_dict[type]}"
             use_sim="${use_sim}"
           />
@@ -134,4 +139,7 @@
           value="${dict ([
           ('LDR01', 's1'),
+          ('LDR02', 's2'),
+          ('LDR03', 'a2m12'),
+          ('LDR04', 'a3'),
           ('LDR06', 's3'),
         ])}" />

Commit message: DEVs have presets for components configurations
Signed-off-by: Jakub Delicat <jakub.delicat@husarion.com>

File: urdf/components.urdf.xacro (robot description, xacro)
@@ -20,9 +20,5 @@
       <xacro:property name="component" value="${config['components'][index]}" scope="parent" />
       <xacro:property name="type" value="${component['type']}" scope="parent" />
-      <xacro:property name="parent_link" value="${component['parent_link']}" scope="parent" />
       <xacro:property name="ns" value="${robot_namespace}" scope="parent" />
-      <xacro:property name="xyz" value="${component['xyz'] if 'xyz' in component else '0.0 0.0 0.0'}" scope="parent" />
-      <xacro:property name="rpy" value="${component['rpy'] if 'rpy' in component else '0.0 0.0 0.0'}" scope="parent" />
-      <xacro:property name="device_ns" value="${component['device_namespace'] if 'device_namespace' in component else ''}" scope="parent" />
       <xacro:property name="dev_models_dict"
         value="${dict ([
@@ -49,4 +45,8 @@
       </xacro:if>
       <xacro:unless value="${type in dev_models_dict}">
+        <xacro:property name="parent_link" value="${component['parent_link']}" scope="parent" />
+        <xacro:property name="xyz" value="${component['xyz'] if 'xyz' in component else '0.0 0.0 0.0'}" scope="parent" />
+        <xacro:property name="rpy" value="${component['rpy'] if 'rpy' in component else '0.0 0.0 0.0'}" scope="parent" />
+        <xacro:property name="device_ns" value="${component['device_namespace'] if 'device_namespace' in component else ''}" scope="parent" />
         <xacro:if value="${type == 'ANT02'}">
           <xacro:include

Commit message: fix dev tf names

File: urdf/components.urdf.xacro (robot description, xacro)
@@ -40,5 +40,4 @@
         />
         <xacro:dev.dev
-          namespace="${ns}"
           model="${dev_models_dict[type]}"
         />

File: urdf/dev.urdf.xacro (robot description, xacro)
@@ -2,6 +2,5 @@
 <robot xmlns:xacro="http://www.ros.org/wiki/xacro">
   <xacro:macro name="dev"
-               params="namespace:=None model:=dev01">
-    <xacro:property name="ns" value="${namespace + '/' if namespace != '' else ''}" />
+               params="model:=dev01">
     <xacro:if value="${model == 'dev01'}">
       <xacro:property name="parent_link" value="body_link" scope="parent" />
@@ -86,10 +85,10 @@
       <xacro:property name="collision_box_xyz"  value="0 0 0.125"      scope="parent" />
     </xacro:if>
-    <joint name="${ns}${model}_joint" type="fixed">
+    <joint name="${model}_joint" type="fixed">
       <origin xyz="${xyz}" rpy="${rpy}" />
       <parent link="${parent_link}" />
-      <child link="${ns}${model}_link" />
+      <child link="${model}_link" />
     </joint>
-    <link name="${ns}${model}_link">
+    <link name="${model}_link">
       <visual>
         <origin xyz="0 0 0" rpy="0 0 0" />
